Commit message: camera orientation fix

File: urdf/hhfc/urdf/hhfc.urdf (robot description, URDF)
Before this commit: robot hhfc, 16 links, 15 joints
Links:
- link camera_link: geometry visual box size=0.1 0.02 0.02
Joints:
- joint camera_joint: origin xyz=0.1 0.0 0.0 rpy=0 0.3490658503988659 0 -> xyz=0.1 0.0 0.0 rpy=-1.9198621771937625 0.0 -1.57079632679489661923

Commit message: update

File: urdf/hhfc/urdf/hhfc.urdf (robot description, URDF)
Before this commit: robot hhfc, 16 links, 15 joints
Joints:
- joint Lleg_ankle_p_joint: limit lower=-0.6981317007977318 upper=0.6981317007977318 effort=100 velocity=5000 -> lower=-0.6981317007977318 upper=0.6981317007977318 effort=100 velocity=15
- joint Lleg_ankle_r_joint: limit lower=-0.3490658503988659 upper=0.3490658503988659 effort=100 velocity=5000 -> lower=-0.3490658503988659 upper=0.3490658503988659 effort=100 velocity=15
- joint Lleg_hip_p_joint: limit lower=-1.5708 upper=3.1416 effort=250 velocity=5000 -> lower=-1.5708 upper=3.1416 effort=250 velocity=20
- joint Lleg_hip_r_joint: limit lower=-0.12217 upper=0.52359 effort=100 velocity=5000 -> lower=-0.12217 upper=0.52359 effort=100 velocity=15
- joint Lleg_hip_y_joint: limit lower=-1.0472 upper=1.2217 effort=100 velocity=5000 -> lower=-1.0472 upper=1.2217 effort=100 velocity=20
- joint Lleg_knee_joint: limit lower=-1.5708 upper=0 effort=250 velocity=5000 -> lower=-1.5708 upper=0 effort=250 velocity=15
- joint Rleg_ankle_p_joint: limit lower=-0.6981317007977318 upper=0.6981317007977318 effort=100 velocity=5000 -> lower=-0.6981317007977318 upper=0.6981317007977318 effort=100 velocity=15
- joint Rleg_ankle_r_joint: limit lower=-0.3490658503988659 upper=0.3490658503988659 effort=100 velocity=5000 -> lower=-0.3490658503988659 upper=0.3490658503988659 effort=100 velocity=15
- joint Rleg_hip_p_joint: limit lower=-1.5708 upper=3.1416 effort=250 velocity=5000 -> lower=-1.5708 upper=3.1416 effort=250 velocity=20
- joint Rleg_hip_r_joint: limit lower=-0.52359 upper=0.12217 effort=100 velocity=5000 -> lower=-0.52359 upper=0.12217 effort=100 velocity=20
- joint Rleg_hip_y_joint: limit lower=-1.2217 upper=1.0472 effort=100 velocity=5000 -> lower=-1.2217 upper=1.0472 effort=100 velocity=20
- joint Rleg_knee_joint: limit lower=-1.5708 upper=0 effort=250 velocity=5000 -> lower=-1.5708 upper=0 effort=250 velocity=15
- joint camera_joint: origin xyz=0.1 0.0 0.0 rpy=-1.9198621771937625 0.0 -1.57079632679489661923 -> xyz=0.1 0.0 0.0 rpy=-2.181661564992912 0.0 -1.57079632679489661923
